Commit message: Fixed URDF and augmented launch files. Added a new launch file for the non-move_base navigation planner. Also changed base_local_planner settings to more closely follow the global path.

File: ros_arduino_python/config/prsg2_description.xacro (robot description, xacro)
@@ -1,4 +1,5 @@
 <?xml version="1.0" encoding="UTF-8" ?>
 <robot name="prsg2_robot" xmlns:xacro="http://www.ros.org/wiki/xacro">
+  <xacro:property name="pi" value="3.14159" />
   <xacro:property name="degree" value="${pi / 180}" />
   <xacro:property name="inch" value="0.0254" />
@@ -16,5 +17,5 @@
   <xacro:property name="camera_setback" value="0.025" />
   <xacro:macro name="material_color" params="r g b a:=1.0">
-    <material>
+    <material name="color_${r}_${g}_${b}_{$a}">
       <color rgba="${r} ${g} ${b} ${a}" />
     </material>
